File: kicad/F-Register.sch (KiCad schematic (older format))
At the start: 10 parts, among them U63 74LS245, U64 74LS173

Commit message: Work on todo list
Parts:
- renumbered D98 to D34, D99 to D35, D100 to D36, D101 to D37, R104 to R40, R105 to R41, R106 to R42, R107 to R43, U63 to U103, U64 to U104
Connections:
- net F_3 renamed PF
- net ~F0~ renamed ~FO~
- net ~F1~ renamed ~FI~
Changed lines of the file:
@@
 $Descr USLetter 11000 8500
 encoding utf-8
-Sheet 22 22
+Sheet 26 26
 Title "Flags Register"
 Date "2019-09-26"
@@
 $EndDescr
 Text HLabel 9550 2950 2    50   Input ~ 0
-~F1~
+~FI~
 Wire Wire Line
 	7500 2650 7500 3050
@@
 AR Path="/5D9E93FA/5DA6F92D" Ref="#PWR?"  Part="1"
 AR Path="/5DA98D6D/5DA9AAB9/5DA6F92D" Ref="#PWR?"  Part="1"
-AR Path="/5DA9DA3D/5DA6F92D" Ref="#PWR?"  Part="1"
-F 0 "#PWR?" H 7600 2200 50  0001 C CNN
+AR Path="/5DA9DA3D/5DA6F92D" Ref="#PWR026"  Part="1"
+F 0 "#PWR026" H 7600 2200 50  0001 C CNN
 F 1 "GND" H 7605 2277 50  0000 C CNN
 F 2 "" H 7600 2450 50  0001 C CNN
@@
 AR Path="/5D9E93FA/5DA6F90E" Ref="#PWR?"  Part="1"
 AR Path="/5DA98D6D/5DA9AAB9/5DA6F90E" Ref="#PWR?"  Part="1"
-AR Path="/5DA9DA3D/5DA6F90E" Ref="#PWR?"  Part="1"
-F 0 "#PWR?" H 3300 4050 50  0001 C CNN
+AR Path="/5DA9DA3D/5DA6F90E" Ref="#PWR027"  Part="1"
+F 0 "#PWR027" H 3300 4050 50  0001 C CNN
 F 1 "VCC" H 3318 4373 50  0000 C CNN
 F 2 "" H 3300 4200 50  0001 C CNN
@@
 	3400 4400 3400 4050
 Text HLabel 3400 4400 3    50   Input ~ 0
-~F0~
+~FO~
 Wire Wire Line
 	8100 4050 8100 5350
@@
 	7800 4050 7800 5050
 Text HLabel 1300 2150 0    50   Output ~ 0
-F_3
+PF
 Text HLabel 1300 2050 0    50   Output ~ 0
 SF
@@
 AR Path="/5D9E93FA/5DA6F8D2" Ref="#PWR?"  Part="1"
 AR Path="/5DA98D6D/5DA9AAB9/5DA6F8D2" Ref="#PWR?"  Part="1"
-AR Path="/5DA9DA3D/5DA6F8D2" Ref="#PWR?"  Part="1"
-F 0 "#PWR?" H 4850 7000 50  0001 C CNN
+AR Path="/5DA9DA3D/5DA6F8D2" Ref="#PWR028"  Part="1"
+F 0 "#PWR028" H 4850 7000 50  0001 C CNN
 F 1 "GND" H 4855 7077 50  0000 C CNN
 F 2 "" H 4850 7250 50  0001 C CNN
@@
 AR Path="/5D9E93FA/5DA6F8C4" Ref="R?"  Part="1"
 AR Path="/5DA98D6D/5DA9AAB9/5DA6F8C4" Ref="R?"  Part="1"
-AR Path="/5DA9DA3D/5DA6F8C4" Ref="R107"  Part="1"
-F 0 "R107" H 5970 6646 50  0000 L CNN
+AR Path="/5DA9DA3D/5DA6F8C4" Ref="R43"  Part="1"
+F 0 "R43" H 5970 6646 50  0000 L CNN
 F 1 "220" H 5970 6555 50  0000 L CNN
 F 2 "" V 5830 6600 50  0001 C CNN
@@
 AR Path="/5D9E93FA/5DA6F8BE" Ref="R?"  Part="1"
 AR Path="/5DA98D6D/5DA9AAB9/5DA6F8BE" Ref="R?"  Part="1"
-AR Path="/5DA9DA3D/5DA6F8BE" Ref="R106"  Part="1"
-F 0 "R106" H 5620 6646 50  0000 L CNN
+AR Path="/5DA9DA3D/5DA6F8BE" Ref="R42"  Part="1"
+F 0 "R42" H 5620 6646 50  0000 L CNN
 F 1 "220" H 5620 6555 50  0000 L CNN
 F 2 "" V 5480 6600 50  0001 C CNN
@@
 AR Path="/5D9E93FA/5DA6F8B8" Ref="R?"  Part="1"
 AR Path="/5DA98D6D/5DA9AAB9/5DA6F8B8" Ref="R?"  Part="1"
-AR Path="/5DA9DA3D/5DA6F8B8" Ref="R105"  Part="1"
-F 0 "R105" H 5270 6646 50  0000 L CNN
+AR Path="/5DA9DA3D/5DA6F8B8" Ref="R41"  Part="1"
+F 0 "R41" H 5270 6646 50  0000 L CNN
 F 1 "220" H 5270 6555 50  0000 L CNN
 F 2 "" V 5130 6600 50  0001 C CNN
@@
 AR Path="/5D9E93FA/5DA6F8B2" Ref="R?"  Part="1"
 AR Path="/5DA98D6D/5DA9AAB9/5DA6F8B2" Ref="R?"  Part="1"
-AR Path="/5DA9DA3D/5DA6F8B2" Ref="R104"  Part="1"
-F 0 "R104" H 4920 6646 50  0000 L CNN
+AR Path="/5DA9DA3D/5DA6F8B2" Ref="R40"  Part="1"
+F 0 "R40" H 4920 6646 50  0000 L CNN
 F 1 "220" H 4920 6555 50  0000 L CNN
 F 2 "" V 4780 6600 50  0001 C CNN
@@
 AR Path="/5D9E93FA/5DA6F87E" Ref="D?"  Part="1"
 AR Path="/5DA98D6D/5DA9AAB9/5DA6F87E" Ref="D?"  Part="1"
-AR Path="/5DA9DA3D/5DA6F87E" Ref="D101"  Part="1"
-F 0 "D101" V 5939 5933 50  0000 R CNN
+AR Path="/5DA9DA3D/5DA6F87E" Ref="D37"  Part="1"
+F 0 "D37" V 5939 5933 50  0000 R CNN
 F 1 "LED" V 5848 5933 50  0000 R CNN
 F 2 "" H 5900 6050 50  0001 C CNN
@@
 AR Path="/5D9E93FA/5DA6F878" Ref="D?"  Part="1"
 AR Path="/5DA98D6D/5DA9AAB9/5DA6F878" Ref="D?"  Part="1"
-AR Path="/5DA9DA3D/5DA6F878" Ref="D100"  Part="1"
-F 0 "D100" V 5589 5933 50  0000 R CNN
+AR Path="/5DA9DA3D/5DA6F878" Ref="D36"  Part="1"
+F 0 "D36" V 5589 5933 50  0000 R CNN
 F 1 "LED" V 5498 5933 50  0000 R CNN
 F 2 "" H 5550 6050 50  0001 C CNN
@@
 AR Path="/5D9E93FA/5DA6F872" Ref="D?"  Part="1"
 AR Path="/5DA98D6D/5DA9AAB9/5DA6F872" Ref="D?"  Part="1"
-AR Path="/5DA9DA3D/5DA6F872" Ref="D99"  Part="1"
-F 0 "D99" V 5239 5933 50  0000 R CNN
+AR Path="/5DA9DA3D/5DA6F872" Ref="D35"  Part="1"
+F 0 "D35" V 5239 5933 50  0000 R CNN
 F 1 "LED" V 5148 5933 50  0000 R CNN
 F 2 "" H 5200 6050 50  0001 C CNN
@@
 AR Path="/5D9E93FA/5DA6F86C" Ref="D?"  Part="1"
 AR Path="/5DA98D6D/5DA9AAB9/5DA6F86C" Ref="D?"  Part="1"
-AR Path="/5DA9DA3D/5DA6F86C" Ref="D98"  Part="1"
-F 0 "D98" V 4889 5933 50  0000 R CNN
+AR Path="/5DA9DA3D/5DA6F86C" Ref="D34"  Part="1"
+F 0 "D34" V 4889 5933 50  0000 R CNN
 F 1 "LED" V 4798 5933 50  0000 R CNN
 F 2 "" H 4850 6050 50  0001 C CNN
@@
 AR Path="/5D9E93FA/5DA6F82A" Ref="U?"  Part="1"
 AR Path="/5DA98D6D/5DA9AAB9/5DA6F82A" Ref="U?"  Part="1"
-AR Path="/5DA9DA3D/5DA6F82A" Ref="U64"  Part="1"
-F 0 "U64" V 7454 4494 50  0000 L CNN
+AR Path="/5DA9DA3D/5DA6F82A" Ref="U104"  Part="1"
+F 0 "U104" V 7454 4494 50  0000 L CNN
 F 1 "74LS173" V 7545 4494 50  0000 L CNN
 F 2 "" H 7500 3550 50  0001 C CNN
@@
 AR Path="/5D9E93FA/5DA6F7FD" Ref="U?"  Part="1"
 AR Path="/5DA98D6D/5DA9AAB9/5DA6F7FD" Ref="U?"  Part="1"
-AR Path="/5DA9DA3D/5DA6F7FD" Ref="U63"  Part="1"
-F 0 "U63" V 2946 2706 50  0000 R CNN
+AR Path="/5DA9DA3D/5DA6F7FD" Ref="U103"  Part="1"
+F 0 "U103" V 2946 2706 50  0000 R CNN
 F 1 "74LS245" V 2855 2706 50  0000 R CNN
 F 2 "" H 2900 3550 50  0001 C CNN
