File: kicad/ALU-A.sch (KiCad schematic (older format))
At the start: 13 parts

Commit message: Work on todo list
Parts:
- removed U? (x2): 74LS194, symbol 74xx:74LS194
- removed U? (x9): 74LS86, symbol 74xx:74LS86
- removed U? (x2): 74LS283, symbol 74xx:74LS283
