File: kicad/ALU-Shift.sch (KiCad schematic (older format))
At the start: 10 parts, among them U100 74LS245, U101 74LS32, U102 74LS86, U93 74LS86, U94 74LS32, U95 74LS32, U96 74LS194, U97 74LS194, U98 74LS02, U99 74LS86

Commit message: Reorganize part references
Parts:
- renumbered U94 to U43, U95 to U43, U101 to U43, U93 to U44, U99 to U44, U102 to U44, U96 to U45, U98 to U46, U97 to U47, U100 to U48
Connections:
- net A_0: now also U44.9; no longer U44.1
- net A_7: now also U43.4, U44.4; no longer U43.1, U44.1
- net CO: now also U43.8; no longer U43.3
- net RL: now also U44.5; no longer U44.2
- net RR: now also U44.10; no longer U44.2
- net at U47.2 (Dsr): now also U43.6; no longer U43.3
- net at U43.2, U44.3: now also U43.5; no longer U43.2
- new net: U43.10, U44.6
- new net: U43.9, U44.8
Changed lines of the file:
@@
 $Descr A4 11693 8268
 encoding utf-8
-Sheet 22 26
+Sheet 11 26
 Title ""
 Date "2019-10-03"
@@
 AR Path="/5E5B2E62/5DF0EA60" Ref="U?"  Part="1"
 AR Path="/5E5B2E62/5E0141CE/5DF0EA60" Ref="U?"  Part="1"
-AR Path="/5E5B2E62/5E0141CE/5DF0B9F6/5DF0EA60" Ref="U97"  Part="1"
-F 0 "U97" H 5950 4481 50  0000 C CNN
+AR Path="/5E5B2E62/5E0141CE/5DF0B9F6/5DF0EA60" Ref="U47"  Part="1"
+F 0 "U47" H 5950 4481 50  0000 C CNN
 F 1 "74LS194" H 5950 4390 50  0000 C CNN
 F 2 "" H 5950 3400 50  0001 C CNN
@@
 AR Path="/5E5B2E62/5DF0EA66" Ref="U?"  Part="1"
 AR Path="/5E5B2E62/5E0141CE/5DF0EA66" Ref="U?"  Part="1"
-AR Path="/5E5B2E62/5E0141CE/5DF0B9F6/5DF0EA66" Ref="U96"  Part="1"
-F 0 "U96" H 3750 4481 50  0000 C CNN
+AR Path="/5E5B2E62/5E0141CE/5DF0B9F6/5DF0EA66" Ref="U45"  Part="1"
+F 0 "U45" H 3750 4481 50  0000 C CNN
 F 1 "74LS194" H 3750 4390 50  0000 C CNN
 F 2 "" H 3750 3400 50  0001 C CNN
@@
 	3250 2800 3250 2900
 $Comp
-L 74xx:74LS86 U93
+L 74xx:74LS86 U44
 U 1 1 5DF678BA
 P 7450 1600
-F 0 "U93" H 7450 1283 50  0000 C CNN
+F 0 "U44" H 7450 1283 50  0000 C CNN
 F 1 "74LS86" H 7450 1374 50  0000 C CNN
 F 2 "" H 7450 1600 50  0001 C CNN
@@
 	3450 1850 3450 2900
 $Comp
-L 74xx:74LS32 U94
+L 74xx:74LS32 U43
 U 1 1 5E065035
 P 3750 2400
-F 0 "U94" V 3704 2588 50  0000 L CNN
+F 0 "U43" V 3704 2588 50  0000 L CNN
 F 1 "74LS32" V 3795 2588 50  0000 L CNN
 F 2 "" H 3750 2400 50  0001 C CNN
@@
 	3650 1600 3650 2100
 $Comp
-L 74xx:74LS32 U95
-U 1 1 5E091AB1
+L 74xx:74LS32 U43
+U 2 1 5E091AB1
 P 6050 2400
-F 0 "U95" V 6004 2588 50  0000 L CNN
+F 0 "U43" V 6004 2588 50  0000 L CNN
 F 1 "74LS32" V 6095 2588 50  0000 L CNN
 F 2 "" H 6050 2400 50  0001 C CNN
 F 3 "http://www.ti.com/lit/gpn/sn74LS32" H 6050 2400 50  0001 C CNN
-	1    6050 2400
+	2    6050 2400
 	0    1    1    0
 $EndComp
@@
 CO
 $Comp
-L 74xx:74LS32 U101
-U 1 1 5E0B4DCA
+L 74xx:74LS32 U43
+U 3 1 5E0B4DCA
 P 2300 4900
-F 0 "U101" H 2300 4583 50  0000 C CNN
+F 0 "U43" H 2300 4583 50  0000 C CNN
 F 1 "74LS32" H 2300 4674 50  0000 C CNN
 F 2 "" H 2300 4900 50  0001 C CNN
 F 3 "http://www.ti.com/lit/gpn/sn74LS32" H 2300 4900 50  0001 C CNN
-	1    2300 4900
+	3    2300 4900
 	-1   0    0    1
 $EndComp
@@
 	2000 4900 1900 4900
 $Comp
-L 74xx:74LS86 U99
-U 1 1 5E0BDF76
+L 74xx:74LS86 U44
+U 2 1 5E0BDF76
 P 3100 4600
-F 0 "U99" H 3100 4283 50  0000 C CNN
+F 0 "U44" H 3100 4283 50  0000 C CNN
 F 1 "74LS86" H 3100 4374 50  0000 C CNN
 F 2 "" H 3100 4600 50  0001 C CNN
 F 3 "74xx/74ls86.pdf" H 3100 4600 50  0001 C CNN
-	1    3100 4600
+	2    3100 4600
 	-1   0    0    1
 $EndComp
@@
 	2700 4800 2600 4800
 $Comp
-L 74xx:74LS86 U102
-U 1 1 5E0C532F
+L 74xx:74LS86 U44
+U 3 1 5E0C532F
 P 3100 5200
-F 0 "U102" H 3100 4883 50  0000 C CNN
+F 0 "U44" H 3100 4883 50  0000 C CNN
 F 1 "74LS86" H 3100 4974 50  0000 C CNN
 F 2 "" H 3100 5200 50  0001 C CNN
 F 3 "74xx/74ls86.pdf" H 3100 5200 50  0001 C CNN
-	1    3100 5200
+	3    3100 5200
 	-1   0    0    1
 $EndComp
@@
 AR Path="/5E5B2E62/5E164880" Ref="U?"  Part="1"
 AR Path="/5E5B2E62/5E0141CE/5D94D587/5E164880" Ref="U?"  Part="1"
-AR Path="/5E5B2E62/5E0141CE/5DF0B9F6/5E164880" Ref="U100"  Part="1"
-F 0 "U100" V 6096 4006 50  0000 R CNN
+AR Path="/5E5B2E62/5E0141CE/5DF0B9F6/5E164880" Ref="U48"  Part="1"
+F 0 "U48" V 6096 4006 50  0000 R CNN
 F 1 "74LS245" V 6005 4006 50  0000 R CNN
 F 2 "" H 6050 4850 50  0001 C CNN
@@
 	5550 4350 5550 4300
 $Comp
-L 74xx:74LS02 U98
+L 74xx:74LS02 U46
 U 1 1 5E1AFD0C
 P 4950 4500
-F 0 "U98" H 4950 4825 50  0000 C CNN
+F 0 "U46" H 4950 4825 50  0000 C CNN
 F 1 "74LS02" H 4950 4734 50  0000 C CNN
 F 2 "" H 4950 4500 50  0001 C CNN
