File: kicad/Control-Logic.sch (KiCad schematic (older format))
At the start: 0 parts

Commit message: Work on todo list
Other:
- note added: "ALU Controls"
- note added: "Register I/O"
- note added: "String together 64k EEPROMS:\nAddress lines: IR_n, CF, ZF, SF, PF, and t-state counter (16 bits)\nOutput lines: Register I/O, ALU controls, etc."
Changed lines of the file:
@@
 $Descr USLetter 11000 8500
 encoding utf-8
-Sheet 21 22
+Sheet 12 26
 Title ""
 Date "2019-09-26"
@@
 Text HLabel 1800 1150 0    50   Output ~ 0
 ~AI~
-Text HLabel 1800 2550 0    50   Input ~ 0
+Text HLabel 2950 2900 0    50   Input ~ 0
 IR_0
-Text HLabel 1800 2650 0    50   Input ~ 0
+Text HLabel 2950 3000 0    50   Input ~ 0
 IR_1
-Text HLabel 1800 2750 0    50   Input ~ 0
+Text HLabel 2950 3100 0    50   Input ~ 0
 IR_2
-Text HLabel 1800 2850 0    50   Input ~ 0
+Text HLabel 2950 3200 0    50   Input ~ 0
 IR_3
-Text HLabel 1800 2950 0    50   Input ~ 0
+Text HLabel 2950 3300 0    50   Input ~ 0
 IR_4
-Text HLabel 1800 3050 0    50   Input ~ 0
+Text HLabel 2950 3400 0    50   Input ~ 0
 IR_5
-Text HLabel 1800 3150 0    50   Input ~ 0
+Text HLabel 2950 3500 0    50   Input ~ 0
 IR_6
-Text HLabel 1800 3250 0    50   Input ~ 0
+Text HLabel 2950 3600 0    50   Input ~ 0
 IR_7
-Text HLabel 1800 4000 0    50   Input ~ 0
-F_3
+Text HLabel 2950 4000 0    50   Input ~ 0
+PF
+Text HLabel 1800 2550 0    50   Output ~ 0
+~TMPO~
+Text HLabel 1800 2650 0    50   Output ~ 0
+~TMPI~
+Text HLabel 1800 2750 0    50   Output ~ 0
+~FO~
+Text HLabel 1800 2850 0    50   Output ~ 0
+~FI~
+Text HLabel 1800 2950 0    50   Output ~ 0
+~IO~
+Text HLabel 1800 3050 0    50   Output ~ 0
+~II~
+Text HLabel 2950 3700 0    50   Input ~ 0
+CF
+Text HLabel 2950 3800 0    50   Input ~ 0
+ZF
+Text HLabel 2950 3900 0    50   Input ~ 0
+SF
+Text HLabel 1800 2450 0    50   Output ~ 0
+~ALUO~
+Text HLabel 1800 3600 0    50   Output ~ 0
+~ADD~
+Text HLabel 1800 3700 0    50   Output ~ 0
+~AND~
+Text HLabel 1800 3800 0    50   Output ~ 0
+~OR~
+Text HLabel 1800 3900 0    50   Output ~ 0
+~XOR~
+Text HLabel 1800 4250 0    50   Output ~ 0
+SUB
+Text HLabel 1800 4350 0    50   Output ~ 0
+RL
+Text HLabel 1800 4450 0    50   Output ~ 0
+RR
+Text HLabel 1800 4000 0    50   Output ~ 0
+~CMP~
+Text HLabel 1800 4100 0    50   Output ~ 0
+~CMPL~
+Text HLabel 1800 4600 0    50   Output ~ 0
+CFENA
 Text HLabel 1800 4700 0    50   Output ~ 0
-~TMPO~
-Text HLabel 1800 4800 0    50   Output ~ 0
-~TMPI~
-Text HLabel 1800 5000 0    50   Output ~ 0
-~FO~
-Text HLabel 1800 5100 0    50   Output ~ 0
-~FI~
-Text HLabel 1800 5300 0    50   Output ~ 0
-~IO~
-Text HLabel 1800 5400 0    50   Output ~ 0
-~II~
-Text HLabel 1800 3700 0    50   Input ~ 0
-CF
-Text HLabel 1800 3800 0    50   Input ~ 0
-ZF
-Text HLabel 1800 3900 0    50   Input ~ 0
-SF
+CFIN
+Text Notes 2550 2500 0    50   ~ 0
+String together 64k EEPROMS:\nAddress lines: IR_n, CF, ZF, SF, PF, and t-state counter (16 bits)\nOutput lines: Register I/O, ALU controls, etc.
+Text HLabel 1800 3150 0    50   Output ~ 0
+~PCO~
+Text HLabel 1800 3250 0    50   Output ~ 0
+~PCI~
+Text HLabel 1800 3350 0    50   Output ~ 0
+~SPO~
+Text HLabel 1800 3450 0    50   Output ~ 0
+~SPI~
+Text HLabel 1800 4850 0    50   Output ~ 0
+INCPC
+Wire Notes Line
+	1850 1000 1400 1000
+Wire Notes Line
+	1400 1000 1400 3500
+Wire Notes Line
+	1400 3500 1850 3500
+Wire Notes Line
+	1850 3500 1850 1000
+Text Notes 1400 3500 1    50   ~ 0
+Register I/O
+Wire Notes Line
+	1850 4750 1850 3550
+Wire Notes Line
+	1850 3550 1400 3550
+Wire Notes Line
+	1400 3550 1400 4750
+Wire Notes Line
+	1400 4750 1850 4750
+Text Notes 1400 4750 1    50   ~ 0
+ALU Controls
 $EndSCHEMATC

Commit message: Finish todo list
Parts:
- added U?: 74LS161, symbol 74xx:74LS161
- added U? (x5): 29F010-TSOP-SP, symbol Memory_Flash:29F010-TSOP-SP
Connections:
- net CF: now also U?.3 (A8), U?.3 (A8), U?.3 (A8), U?.3 (A8), U?.3 (A8)
- net CFENA: now also U?.23 (D2)
- net CFIN: now also U?.25 (D3)
- net INCPC: now also U?.26 (D4)
- net IR_0: now also U?.20 (A0), U?.20 (A0), U?.20 (A0), U?.20 (A0), U?.20 (A0)
- net IR_1: now also U?.19 (A1), U?.19 (A1), U?.19 (A1), U?.19 (A1), U?.19 (A1)
- net IR_2: now also U?.18 (A2), U?.18 (A2), U?.18 (A2), U?.18 (A2), U?.18 (A2)
- net IR_3: now also U?.17 (A3), U?.17 (A3), U?.17 (A3), U?.17 (A3), U?.17 (A3)
- net IR_4: now also U?.16 (A4), U?.16 (A4), U?.16 (A4), U?.16 (A4), U?.16 (A4)
- net IR_5: now also U?.15 (A5), U?.15 (A5), U?.15 (A5), U?.15 (A5), U?.15 (A5)
- net IR_6: now also U?.14 (A6), U?.14 (A6), U?.14 (A6), U?.14 (A6), U?.14 (A6)
- net IR_7: now also U?.13 (A7), U?.13 (A7), U?.13 (A7), U?.13 (A7), U?.13 (A7)
- net PF: now also U?.1 (A11), U?.1 (A11), U?.1 (A11), U?.1 (A11), U?.1 (A11)
- net RL: now also U?.21 (D0)
- net RR: now also U?.22 (D1)
- net SF: now also U?.31 (A10), U?.31 (A10), U?.31 (A10), U?.31 (A10), U?.31 (A10)
- net SUB: now also U?.29 (D7)
- net ZF: now also U?.2 (A9), U?.2 (A9), U?.2 (A9), U?.2 (A9), U?.2 (A9)
- net ~ADD~: now also U?.22 (D1)
- net ~AI~: now also U?.22 (D1)
- net ~ALUO~: now also U?.28 (D6)
- net ~AND~: now also U?.23 (D2)
- net ~AO~: now also U?.21 (D0)
- net ~BI~: now also U?.25 (D3)
- net ~BO~: now also U?.23 (D2)
- net ~CI~: now also U?.27 (D5)
- net ~CMPL~: now also U?.28 (D6)
- net ~CMP~: now also U?.27 (D5)
- net ~CO~: now also U?.26 (D4)
- net ~DI~: now also U?.29 (D7)
- net ~DO~: now also U?.28 (D6)
- net ~EI~: now also U?.22 (D1)
- net ~EO~: now also U?.21 (D0)
- net ~FI~: now also U?.23 (D2)
- net ~FO~: now also U?.22 (D1)
- net ~HI~: now also U?.25 (D3)
- net ~HO~: now also U?.23 (D2)
- net ~II~: now also U?.26 (D4)
- net ~IO~: now also U?.25 (D3)
- net ~LI~: now also U?.27 (D5)
- net ~LO~: now also U?.26 (D4)
- net ~OR~: now also U?.25 (D3)
- net ~PCI~: now also U?.28 (D6)
- net ~PCO~: now also U?.27 (D5)
- net ~SPI~: now also U?.21 (D0)
- net ~SPO~: now also U?.29 (D7)
- net ~TMPI~: now also U?.21 (D0)
- net ~TMPO~: now also U?.29 (D7)
- net ~XOR~: now also U?.26 (D4)
- new net: U?.11 (A15), U?.11 (A15), U?.11 (A15), U?.11 (A15), U?.11 (A15), U?.11 (Q3)
- new net: U?.12 (Q2), U?.5 (A14), U?.5 (A14), U?.5 (A14), U?.5 (A14), U?.5 (A14)
- new net: U?.13 (Q1), U?.4 (A13), U?.4 (A13), U?.4 (A13), U?.4 (A13), U?.4 (A13)
- new net: U?.12 (A12), U?.12 (A12), U?.12 (A12), U?.12 (A12), U?.12 (A12), U?.14 (Q0)
- new net CLK: U?.2 (CP)
- new net DECSP: U?.28 (D6)
- new net GND: U?.10 (A16), U?.10 (A16), U?.10 (A16), U?.10 (A16), U?.10 (A16), U?.3 (D0), U?.4 (D1), U?.5 (D2), U?.6 (D3)
- new net INCSP: U?.27 (D5)
- new net RST: U?.1 (~MR)
- new net VCC: U?.10 (CET), U?.7 (CEP)
- no-connect marks 0 -> 1
Other:
- note removed: "ALU Controls"
- note removed: "Register I/O"
- note removed: "String together 64k EEPROMS:\nAddress lines: IR_n, CF, ZF, SF, PF, and t-state counter (16 bits)\nOutput lines: Register I/O, ALU controls, etc."

Commit message: Reorganize part references
Parts:
- gave numbers to parts that had none: 6
Changed lines of the file:
@@
 DECSP
 $Comp
-L 74xx:74LS161 U?
+L 74xx:74LS161 U50
 U 1 1 5E8FB423
 P 2700 2000
-F 0 "U?" H 2700 2981 50  0000 C CNN
+F 0 "U50" H 2700 2981 50  0000 C CNN
 F 1 "74LS161" H 2700 2890 50  0000 C CNN
 F 2 "" H 2700 2000 50  0001 C CNN
@@
 	3200 1350 3200 1500
 $Comp
-L Memory_Flash:29F010-TSOP-SP U?
+L Memory_Flash:29F010-TSOP-SP U49
 U 1 1 5E904D82
 P 1800 4950
-F 0 "U?" H 1800 6331 50  0000 C CNN
+F 0 "U49" H 1800 6331 50  0000 C CNN
 F 1 "29F010-TSOP-SP" H 1800 6240 50  0000 C CNN
 F 2 "" H 1800 4950 50  0001 C CNN
@@
 	1700 5550 1700 6000
 $Comp
-L Memory_Flash:29F010-TSOP-SP U?
+L Memory_Flash:29F010-TSOP-SP U51
 U 1 1 5E93DAA5
 P 4500 4950
-F 0 "U?" H 4500 6331 50  0000 C CNN
+F 0 "U51" H 4500 6331 50  0000 C CNN
 F 1 "29F010-TSOP-SP" H 4500 6240 50  0000 C CNN
 F 2 "" H 4500 4950 50  0001 C CNN
@@
 	1000 4300 1000 4350
 $Comp
-L Memory_Flash:29F010-TSOP-SP U?
+L Memory_Flash:29F010-TSOP-SP U53
 U 1 1 5E9C71F9
 P 7200 4950
-F 0 "U?" H 7200 6331 50  0000 C CNN
+F 0 "U53" H 7200 6331 50  0000 C CNN
 F 1 "29F010-TSOP-SP" H 7200 6240 50  0000 C CNN
 F 2 "" H 7200 4950 50  0001 C CNN
@@
 	6450 1350 6450 900
 $Comp
-L Memory_Flash:29F010-TSOP-SP U?
+L Memory_Flash:29F010-TSOP-SP U52
 U 1 1 5EB0A972
 P 6550 1950
-F 0 "U?" H 6550 3331 50  0000 C CNN
+F 0 "U52" H 6550 3331 50  0000 C CNN
 F 1 "29F010-TSOP-SP" H 6550 3240 50  0000 C CNN
 F 2 "" H 6550 1950 50  0001 C CNN
@@
 	7350 2700 8000 2700
 $Comp
-L Memory_Flash:29F010-TSOP-SP U?
+L Memory_Flash:29F010-TSOP-SP U54
 U 1 1 5EC4C3F0
 P 9250 1950
-F 0 "U?" H 9250 3331 50  0000 C CNN
+F 0 "U54" H 9250 3331 50  0000 C CNN
 F 1 "29F010-TSOP-SP" H 9250 3240 50  0000 C CNN
 F 2 "" H 9250 1950 50  0001 C CNN
