File: breadboard-computer-video/Horizontal_Generator.sch (KiCad schematic (older format))
At the start: 3 parts

Commit message: Finished H and V generators
Parts:
- added U? (x4): 74LS21, symbol 74xx:74LS21
- added U? (x4): 74LS32, symbol 74xx:74LS32
- added U? (x4): 74LS04, symbol 74xx:74LS04
- added U?: 74LS08, symbol 74xx:74LS08
Connections:
- net labels added: H_Blank, H_Sync
- wire segments 5 -> 59

Commit message: Finished sync generation, added pixel clock
Parts:
- removed U? (x3): 74LS168, symbol 74xx:74LS168
- added U? (x3): 74LS161, symbol 74xx:74LS161
- added U?: 74LS30, symbol 74xx:74LS30
- added U? (x2): 74LS04, symbol 74xx:74LS04
Connections:
- net labels added: LINE
- wire segments 59 -> 130

Commit message: finished
Parts:
- removed U? (x3): 74LS161, symbol 74xx:74LS161
- added U? (x3): 74LS163, symbol 74xx:74LS163
Connections:
- net CP: now also U?.2 (CP), U?.2 (CP), U?.2 (CP)
- net LINE: now also U?.1 (~MR), U?.1 (~MR), U?.1 (~MR)
- net VCC: now also U?.10 (CET), U?.16 (VCC), U?.16 (VCC), U?.16 (VCC), U?.7 (CEP), U?.7 (CEP), U?.7 (CEP), U?.9 (~PE), U?.9 (~PE), U?.9 (~PE)
- net at U?.1, U?.11: now also U?.14 (Q0)
- net at U?.1, U?.2: now also U?.13 (Q1)
- net at U?.4: now also U?.12 (Q2)
- net at U?.5: now also U?.11 (Q3)
- net at U?.10, U?.13, U?.9: now also U?.14 (Q0)
- net at U?.12, U?.3, U?.4: now also U?.13 (Q1)
- net at U?.1, U?.13: now also U?.12 (Q2)
- net at U?.2, U?.4, U?.5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: now also U?.11 (Q3)
- net at U?.11, U?.12, U?.13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: now also U?.14 (Q0)
- new net: U?.10 (CET), U?.15 (TC) (x2)
- new net Earth: U?.8 (GND), U?.8 (GND), U?.8 (GND)
Changed lines of the file:
@@
 $Descr A4 11693 8268
 encoding utf-8
-Sheet 3 4
+Sheet 3 5
 Title ""
 Date ""
@@
 Comment4 ""
 $EndDescr
-Text HLabel 8350 6050 3    50   Input ~ 0
+Text HLabel 8350 6300 3    50   Input ~ 0
 CP
 Wire Wire Line
 	3350 5650 3350 6050
-$Comp
-L power:GND #PWR?
-U 1 1 5DBA5B33
-P 6350 5150
-F 0 "#PWR?" H 6350 4900 50  0001 C CNN
-F 1 "GND" V 6355 5022 50  0000 R CNN
-F 2 "" H 6350 5150 50  0001 C CNN
-F 3 "" H 6350 5150 50  0001 C CNN
-	1    6350 5150
-	0    -1   -1   0
-$EndComp
-$Comp
-L power:GND #PWR?
-U 1 1 5DBA5B39
-P 3850 5150
-F 0 "#PWR?" H 3850 4900 50  0001 C CNN
-F 1 "GND" V 3855 5022 50  0000 R CNN
-F 2 "" H 3850 5150 50  0001 C CNN
-F 3 "" H 3850 5150 50  0001 C CNN
-	1    3850 5150
-	0    -1   -1   0
-$EndComp
-$Comp
-L power:GND #PWR?
-U 1 1 5DBAB347
-P 8850 5150
-F 0 "#PWR?" H 8850 4900 50  0001 C CNN
-F 1 "GND" V 8855 5022 50  0000 R CNN
-F 2 "" H 8850 5150 50  0001 C CNN
-F 3 "" H 8850 5150 50  0001 C CNN
-	1    8850 5150
-	0    -1   -1   0
-$EndComp
 Wire Wire Line
 	5850 5650 5850 6050
@@
 Text HLabel 6650 2050 1    50   Output ~ 0
 H_Sync
-$Comp
-L 74xx:74LS161 U?
-U 1 1 5DB5E3FC
-P 5550 5150
-F 0 "U?" V 5596 4306 50  0000 R CNN
-F 1 "74LS161" V 5505 4306 50  0000 R CNN
-F 2 "" H 5550 5150 50  0001 C CNN
-F 3 "http://www.ti.com/lit/gpn/sn74LS161" H 5550 5150 50  0001 C CNN
-	1    5550 5150
-	0    -1   -1   0
-$EndComp
-$Comp
-L 74xx:74LS161 U?
-U 1 1 5DB6099E
-P 3050 5150
-F 0 "U?" V 3096 4306 50  0000 R CNN
-F 1 "74LS161" V 3005 4306 50  0000 R CNN
-F 2 "" H 3050 5150 50  0001 C CNN
-F 3 "http://www.ti.com/lit/gpn/sn74LS161" H 3050 5150 50  0001 C CNN
-	1    3050 5150
-	0    -1   -1   0
-$EndComp
-$Comp
-L 74xx:74LS161 U?
-U 1 1 5DB5CF73
-P 8050 5150
-F 0 "U?" V 8096 4306 50  0000 R CNN
-F 1 "74LS161" V 8005 4306 50  0000 R CNN
-F 2 "" H 8050 5150 50  0001 C CNN
-F 3 "http://www.ti.com/lit/gpn/sn74LS161" H 8050 5150 50  0001 C CNN
-	1    8050 5150
-	0    -1   -1   0
-$EndComp
 Wire Wire Line
 	8350 5650 8350 6050
@@
 Wire Wire Line
 	5350 5750 6050 5750
+$Comp
+L 74xx:74LS163 U?
+U 1 1 5E152224
+P 3050 5150
+F 0 "U?" V 3096 4306 50  0000 R CNN
+F 1 "74LS163" V 3005 4306 50  0000 R CNN
+F 2 "" H 3050 5150 50  0001 C CNN
+F 3 "http://www.ti.com/lit/gpn/sn74LS163" H 3050 5150 50  0001 C CNN
+	1    3050 5150
+	0    -1   -1   0
+$EndComp
+$Comp
+L 74xx:74LS163 U?
+U 1 1 5E1579F5
+P 5550 5150
+F 0 "U?" V 5596 4306 50  0000 R CNN
+F 1 "74LS163" V 5505 4306 50  0000 R CNN
+F 2 "" H 5550 5150 50  0001 C CNN
+F 3 "http://www.ti.com/lit/gpn/sn74LS163" H 5550 5150 50  0001 C CNN
+	1    5550 5150
+	0    -1   -1   0
+$EndComp
+$Comp
+L 74xx:74LS163 U?
+U 1 1 5E15D181
+P 8050 5150
+F 0 "U?" V 8096 4306 50  0000 R CNN
+F 1 "74LS163" V 8005 4306 50  0000 R CNN
+F 2 "" H 8050 5150 50  0001 C CNN
+F 3 "http://www.ti.com/lit/gpn/sn74LS163" H 8050 5150 50  0001 C CNN
+	1    8050 5150
+	0    -1   -1   0
+$EndComp
+Wire Wire Line
+	8850 5150 8850 6150
+Wire Wire Line
+	8850 6150 6350 6150
+Wire Wire Line
+	6350 5150 6350 6150
+Connection ~ 6350 6150
+Wire Wire Line
+	6350 6150 3850 6150
+Wire Wire Line
+	3850 5150 3850 6150
+Connection ~ 3850 6150
+Wire Wire Line
+	3850 6150 1800 6150
+Wire Wire Line
+	8350 6050 8350 6300
+Connection ~ 8350 6050
+$Comp
+L power:Earth #PWR?
+U 1 1 5E1A3868
+P 1800 6150
+F 0 "#PWR?" H 1800 5900 50  0001 C CNN
+F 1 "Earth" H 1800 6000 50  0001 C CNN
+F 2 "" H 1800 6150 50  0001 C CNN
+F 3 "~" H 1800 6150 50  0001 C CNN
+	1    1800 6150
+	0    1    1    0
+$EndComp
 $EndSCHEMATC

Commit message: fixed labels
Parts:
- gave numbers to parts that had none: 12
Changed lines of the file:
@@
 	5850 5650 5850 6050
 $Comp
-L 74xx:74LS21 U?
+L 74xx:74LS21 U21
 U 1 1 5D97D00C
 P 5200 4100
-F 0 "U?" V 5246 3895 50  0000 R CNN
+F 0 "U21" V 5246 3895 50  0000 R CNN
 F 1 "74LS21" V 5155 3895 50  0000 R CNN
 F 2 "" H 5200 4100 50  0001 C CNN
@@
 	5050 4650 5050 4500
 $Comp
-L 74xx:74LS21 U?
+L 74xx:74LS21 U16
 U 2 1 5D980DC0
 P 2600 4100
-F 0 "U?" V 2646 3895 50  0000 R CNN
+F 0 "U16" V 2646 3895 50  0000 R CNN
 F 1 "74LS21" V 2555 3895 50  0000 R CNN
 F 2 "" H 2600 4100 50  0001 C CNN
@@
 	2550 4550 2550 4650
 $Comp
-L 74xx:74LS32 U?
+L 74xx:74LS32 U17
 U 1 1 5D985BC0
 P 2700 3500
-F 0 "U?" V 2746 3320 50  0000 R CNN
+F 0 "U17" V 2746 3320 50  0000 R CNN
 F 1 "74LS32" V 2655 3320 50  0000 R CNN
 F 2 "" H 2700 3500 50  0001 C CNN
@@
 	2800 4250 2800 3800
 $Comp
-L 74xx:74LS32 U?
+L 74xx:74LS32 U17
 U 2 1 5D98B302
 P 7450 3500
-F 0 "U?" V 7496 3320 50  0000 R CNN
+F 0 "U17" V 7496 3320 50  0000 R CNN
 F 1 "74LS32" V 7405 3320 50  0000 R CNN
 F 2 "" H 7450 3500 50  0001 C CNN
@@
 	7350 3800 6850 3800
 $Comp
-L 74xx:74LS21 U?
+L 74xx:74LS21 U16
 U 1 1 5D992A54
 P 4050 3600
-F 0 "U?" V 4096 3395 50  0000 R CNN
+F 0 "U16" V 4096 3395 50  0000 R CNN
 F 1 "74LS21" V 4005 3395 50  0000 R CNN
 F 2 "" H 4050 3600 50  0001 C CNN
@@
 $EndComp
 $Comp
-L 74xx:74LS04 U?
+L 74xx:74LS04 U13
 U 1 1 5D998351
 P 3600 3900
-F 0 "U?" H 3600 4217 50  0000 C CNN
+F 0 "U13" H 3600 4217 50  0000 C CNN
 F 1 "74LS04" H 3600 4126 50  0000 C CNN
 F 2 "" H 3600 3900 50  0001 C CNN
@@
 $EndComp
 $Comp
-L 74xx:74LS04 U?
+L 74xx:74LS04 U13
 U 2 1 5D999D2D
 P 3700 4300
-F 0 "U?" H 3700 4617 50  0000 C CNN
+F 0 "U13" H 3700 4617 50  0000 C CNN
 F 1 "74LS04" H 3700 4526 50  0000 C CNN
 F 2 "" H 3700 4300 50  0001 C CNN
@@
 	4100 4100 4100 4200
 $Comp
-L 74xx:74LS08 U?
+L 74xx:74LS08 U23
 U 1 1 5D9C29E1
 P 6750 2950
-F 0 "U?" V 6796 2770 50  0000 R CNN
+F 0 "U23" V 6796 2770 50  0000 R CNN
 F 1 "74LS08" V 6705 2770 50  0000 R CNN
 F 2 "" H 6750 2950 50  0001 C CNN
@@
 $EndComp
 $Comp
-L 74xx:74LS04 U?
+L 74xx:74LS04 U19
 U 3 1 5D9D9387
 P 4800 3600
-F 0 "U?" V 4846 3420 50  0000 R CNN
+F 0 "U19" V 4846 3420 50  0000 R CNN
 F 1 "74LS04" V 4755 3420 50  0000 R CNN
 F 2 "" H 4800 3600 50  0001 C CNN
@@
 $EndComp
 $Comp
-L 74xx:74LS04 U?
+L 74xx:74LS04 U13
 U 4 1 5D9F290B
 P 5350 3000
-F 0 "U?" V 5396 2820 50  0000 R CNN
+F 0 "U13" V 5396 2820 50  0000 R CNN
 F 1 "74LS04" V 5305 2820 50  0000 R CNN
 F 2 "" H 5350 3000 50  0001 C CNN
@@
 $EndComp
 $Comp
-L 74xx:74LS21 U?
+L 74xx:74LS21 U21
 U 2 1 5DA0BF5D
 P 5400 2050
-F 0 "U?" V 5446 1845 50  0000 R CNN
+F 0 "U21" V 5446 1845 50  0000 R CNN
 F 1 "74LS21" V 5355 1845 50  0000 R CNN
 F 2 "" H 5400 2050 50  0001 C CNN
@@
 	4100 4200 4100 4600
 $Comp
-L 74xx:74LS32 U?
+L 74xx:74LS32 U3
 U 2 1 5DA522B7
 P 4450 3000
-F 0 "U?" V 4496 2820 50  0000 R CNN
+F 0 "U3" V 4496 2820 50  0000 R CNN
 F 1 "74LS32" V 4405 2820 50  0000 R CNN
 F 2 "" H 4450 3000 50  0001 C CNN
@@
 	7550 4000 7550 4350
 $Comp
-L 74xx:74LS32 U?
+L 74xx:74LS32 U3
 U 4 1 5DA8F5B6
 P 6650 2350
-F 0 "U?" V 6696 2170 50  0000 R CNN
+F 0 "U3" V 6696 2170 50  0000 R CNN
 F 1 "74LS32" V 6605 2170 50  0000 R CNN
 F 2 "" H 6650 2350 50  0001 C CNN
@@
 LINE
 $Comp
-L 74xx:74LS30 U?
+L 74xx:74LS30 U20
 U 1 1 5DCBD3EC
 P 4950 6500
-F 0 "U?" H 4950 7025 50  0000 C CNN
+F 0 "U20" H 4950 7025 50  0000 C CNN
 F 1 "74LS30" H 4950 6934 50  0000 C CNN
 F 2 "" H 4950 6500 50  0001 C CNN
@@
 	5050 4500 5050 4400
 $Comp
-L 74xx:74LS04 U?
+L 74xx:74LS04 U1
 U 5 1 5DD79FBA
 P 4500 5100
-F 0 "U?" V 4454 5280 50  0000 L CNN
+F 0 "U1" V 4454 5280 50  0000 L CNN
 F 1 "74LS04" V 4545 5280 50  0000 L CNN
 F 2 "" H 4500 5100 50  0001 C CNN
@@
 Connection ~ 3900 3900
 $Comp
-L 74xx:74LS04 U?
+L 74xx:74LS04 U1
 U 6 1 5DDA5C8B
 P 3650 6700
-F 0 "U?" H 3650 7017 50  0000 C CNN
+F 0 "U1" H 3650 7017 50  0000 C CNN
 F 1 "74LS04" H 3650 6926 50  0000 C CNN
 F 2 "" H 3650 6700 50  0001 C CNN
@@
 	5350 5750 6050 5750
 $Comp
-L 74xx:74LS163 U?
+L 74xx:74LS163 U18
 U 1 1 5E152224
 P 3050 5150
-F 0 "U?" V 3096 4306 50  0000 R CNN
+F 0 "U18" V 3096 4306 50  0000 R CNN
 F 1 "74LS163" V 3005 4306 50  0000 R CNN
 F 2 "" H 3050 5150 50  0001 C CNN
@@
 $EndComp
 $Comp
-L 74xx:74LS163 U?
+L 74xx:74LS163 U22
 U 1 1 5E1579F5
 P 5550 5150
-F 0 "U?" V 5596 4306 50  0000 R CNN
+F 0 "U22" V 5596 4306 50  0000 R CNN
 F 1 "74LS163" V 5505 4306 50  0000 R CNN
 F 2 "" H 5550 5150 50  0001 C CNN
@@
 $EndComp
 $Comp
-L 74xx:74LS163 U?
+L 74xx:74LS163 U24
 U 1 1 5E15D181
 P 8050 5150
-F 0 "U?" V 8096 4306 50  0000 R CNN
+F 0 "U24" V 8096 4306 50  0000 R CNN
 F 1 "74LS163" V 8005 4306 50  0000 R CNN
 F 2 "" H 8050 5150 50  0001 C CNN

Commit message: various things
Parts:
- removed U1, U13, U19: 74LS04, symbol 74xx:74LS04
- removed U16, U21: 74LS21, symbol 74xx:74LS21
- removed U17, U3: 74LS32, symbol 74xx:74LS32
- removed U20: 74LS30, symbol 74xx:74LS30
- removed U23: 74LS08, symbol 74xx:74LS08
- added U? (x4): 74LS02, symbol 74xx:74LS02
- added U? (x7): 74LS08, symbol 74xx:74LS08
- added U?: 74LS04, symbol 74xx:74LS04
Connections:
- net VCC is gone; now on an unnamed net: U18.10 (CET), U18.16 (VCC), U18.7 (CEP), U18.9 (~PE), U22.16 (VCC), U22.7 (CEP), U22.9 (~PE), U24.16 (VCC), U24.7 (CEP), U24.9 (~PE)
- net CP: no longer U22.2 (CP), U24.2 (CP)
- net H_Blank: now also U?.13, U?.13
- net H_Sync: now also U?.11
- net LINE: no longer U18.1 (~MR), U22.1 (~MR), U24.1 (~MR)
- net at U22.14 (Q0): now also U?.10
- net at U22.12 (Q2): now also U?.5
- net at U22.11 (Q3): now also U?.4
- net at U18.13 (Q1): now also U?.1, U?.9, U?.9
- net at U18.11 (Q3): now also U?.2
- net at U24.14 (Q0): now also U?.1
- net at U22.10 (CET): now also U24.10 (CET); no longer U18.15 (TC)
- net at U22.15 (TC): now also U24.2 (CP); no longer U24.10 (CET)
- net at U24.13 (Q1): now also U?.2, U?.5
- net Earth: no longer names the net of U18.8 (GND), U22.8 (GND), U24.8 (GND)
- new net: U18.1 (~MR), U22.1 (~MR), U24.1 (~MR), U?.4
- new net: U18.15 (TC), U22.2 (CP)
- new net: U?.1, U?.5
- new net: U?.2, U?.8
- new net: U?.12, U?.3, U?.4
- new net: U?.6, U?.6
- new net: U?.3, U?.4
- new net: U?.3, U?.9
- new net: U?.10, U?.6, U?.8
- new net: U?.3, U?.8
- new net: U?.10, U?.11, U?.12
- no-connect marks 0 -> 13
Other:
- moved on the sheet: U18, U22, U24

Commit message: finished hv sync
Parts:
- added unit 3 of U16
- added unit 1 of U16
- added unit 4 of U17
- added U18: 74LS08, symbol 74xx:74LS08
- gave numbers to parts that had none: 6
- renumbered U18 to U19, U22 to U20, U24 to U21
Connections:
- net H_Blank: now also U16.6; no longer U2.13
- net LINE: now also U16.2
- net at U19.11 (Q3): now also U11.10; no longer U11.2
- net at U19.12 (Q2): now also U11.2
- net at U11.1, U11.9, U15.9: now also U19.14 (Q0), U17.12; no longer U19.13 (Q1)
- net at U20.11 (Q3): now also U15.1; no longer U11.4
- net at U20.12 (Q2): now also U11.4, U18.1, U18.2; no longer U10.5
- net at U20.13 (Q1): now also U10.5
- net at U20.14 (Q0): no longer U11.10
- net at U11.5, U15.2: now also U21.14 (Q0); no longer U21.13 (Q1)
- net at U15.8, U16.3: now also U2.11
- new net: U17.11, U18.3
- new net: U16.5, U17.10
- new net: U17.13, U2.12
- new net: U16.1, U2.13
- no-connect marks 13 -> 18
Other:
- moved on the sheet: U10B, U11A, U11B, U11C, U15A, U15C, U15D, U16B, U17A, U17B, U17C, U19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
