File: breadboard-computer-video/Vertical_Generator.sch (KiCad schematic (older format))
At the start: 10 parts

Commit message: Finished sync generation, added pixel clock
Parts:
- removed U? (x2): 74LS168, symbol 74xx:74LS168
- added U? (x2): 74LS161, symbol 74xx:74LS161
Connections:
- wire segments 39 -> 45
Changed lines of the file:
@@
 $EndDescr
-$Comp
-L 74xx:74LS168 U?
-U 1 1 5D9CF495
-P 4300 4700
-F 0 "U?" V 4346 3756 50  0000 R CNN
-F 1 "74LS168" V 4255 3756 50  0000 R CNN
-F 2 "" H 4300 4700 50  0001 C CNN
-F 3 "http://www.ti.com/lit/gpn/sn74LS168" H 4300 4700 50  0001 C CNN
-	1    4300 4700
-	0    -1   -1   0
-$EndComp
-$Comp
-L 74xx:74LS168 U?
-U 1 1 5D9D01E7
-P 6600 4700
-F 0 "U?" V 6646 3756 50  0000 R CNN
-F 1 "74LS168" V 6555 3756 50  0000 R CNN
-F 2 "" H 6600 4700 50  0001 C CNN
-F 3 "http://www.ti.com/lit/gpn/sn74LS168" H 6600 4700 50  0001 C CNN
-	1    6600 4700
-	0    -1   -1   0
-$EndComp
 $Comp
 L 74xx:74LS08 U?
@@
 Wire Wire Line
 	4100 4200 4000 4200
-Connection ~ 4000 4200
 Wire Wire Line
 	4600 3500 4600 3800
@@
 	0    -1   -1   0
 $EndComp
-Text HLabel 6100 5600 3    50   Input ~ 0
+Text HLabel 6800 5600 3    50   Input ~ 0
 CP
 Text HLabel 3800 2300 1    50   Output ~ 0
@@
 Wire Wire Line
 	3800 2300 3800 2550
-Wire Wire Line
-	4900 5200 4900 5600
-Wire Wire Line
-	4900 5600 7200 5600
-Wire Wire Line
-	7200 5600 7200 5200
 $Comp
 L power:GND #PWR?
 U 1 1 5DB889DE
-P 7500 4700
-F 0 "#PWR?" H 7500 4450 50  0001 C CNN
-F 1 "GND" V 7505 4572 50  0000 R CNN
-F 2 "" H 7500 4700 50  0001 C CNN
-F 3 "" H 7500 4700 50  0001 C CNN
-	1    7500 4700
+P 7300 4700
+F 0 "#PWR?" H 7300 4450 50  0001 C CNN
+F 1 "GND" V 7305 4572 50  0000 R CNN
+F 2 "" H 7300 4700 50  0001 C CNN
+F 3 "" H 7300 4700 50  0001 C CNN
+	1    7300 4700
 	0    -1   -1   0
 $EndComp
@@
 L power:GND #PWR?
 U 1 1 5DB893FF
-P 5200 4700
-F 0 "#PWR?" H 5200 4450 50  0001 C CNN
-F 1 "GND" V 5205 4572 50  0000 R CNN
-F 2 "" H 5200 4700 50  0001 C CNN
-F 3 "" H 5200 4700 50  0001 C CNN
-	1    5200 4700
+P 5000 4700
+F 0 "#PWR?" H 5000 4450 50  0001 C CNN
+F 1 "GND" V 5005 4572 50  0000 R CNN
+F 2 "" H 5000 4700 50  0001 C CNN
+F 3 "" H 5000 4700 50  0001 C CNN
+	1    5000 4700
 	0    -1   -1   0
 $EndComp
@@
 	0    -1   -1   0
 $EndComp
+$Comp
+L 74xx:74LS161 U?
+U 1 1 5DAF5520
+P 6500 4700
+F 0 "U?" V 6546 3856 50  0000 R CNN
+F 1 "74LS161" V 6455 3856 50  0000 R CNN
+F 2 "" H 6500 4700 50  0001 C CNN
+F 3 "http://www.ti.com/lit/gpn/sn74LS161" H 6500 4700 50  0001 C CNN
+	1    6500 4700
+	0    -1   -1   0
+$EndComp
+Wire Wire Line
+	6800 5200 6800 5600
+$Comp
+L 74xx:74LS161 U?
+U 1 1 5DB20441
+P 4200 4700
+F 0 "U?" V 4246 3856 50  0000 R CNN
+F 1 "74LS161" V 4155 3856 50  0000 R CNN
+F 2 "" H 4200 4700 50  0001 C CNN
+F 3 "http://www.ti.com/lit/gpn/sn74LS161" H 4200 4700 50  0001 C CNN
+	1    4200 4700
+	0    -1   -1   0
+$EndComp
+Connection ~ 4000 4200
+Wire Wire Line
+	4500 5200 4500 5600
+Wire Wire Line
+	4500 5600 6800 5600
+Wire Wire Line
+	4700 5200 4700 5400
+Wire Wire Line
+	4700 5400 7000 5400
+Wire Wire Line
+	7000 5400 7000 5200
+Wire Wire Line
+	5800 2200 7750 2200
+Wire Wire Line
+	7750 5400 7000 5400
+Connection ~ 7000 5400
+Wire Wire Line
+	7750 2200 7750 5400
 $EndSCHEMATC

Commit message: finished
Parts:
- removed U? (x2): 74LS161, symbol 74xx:74LS161
- added U? (x2): 74LS163, symbol 74xx:74LS163
Connections:
- net CP: now also U?.2 (CP), U?.2 (CP)
- net GND: now also U?.8 (GND), U?.8 (GND)
- net VCC: now also U?.16 (VCC), U?.16 (VCC)
- net at U?.1, U?.3: now also U?.13 (Q1)
- net at U?.2, U?.5: now also U?.12 (Q2)
- net at U?.3, U?.9: now also U?.11 (Q3)
- net at U?.6: now also U?.14 (Q0)
- net at U?.8: now also U?.1 (~MR), U?.1 (~MR)
- net at U?.1: now also U?.14 (Q0)
- net at U?.5: now also U?.11 (Q3)
- net at U?.4: now also U?.12 (Q2)
Changed lines of the file:
@@
 $Descr A4 11693 8268
 encoding utf-8
-Sheet 2 4
+Sheet 2 5
 Title ""
 Date ""
@@
 	0    -1   -1   0
 $EndComp
-$Comp
-L 74xx:74LS161 U?
-U 1 1 5DAF5520
-P 6500 4700
-F 0 "U?" V 6546 3856 50  0000 R CNN
-F 1 "74LS161" V 6455 3856 50  0000 R CNN
-F 2 "" H 6500 4700 50  0001 C CNN
-F 3 "http://www.ti.com/lit/gpn/sn74LS161" H 6500 4700 50  0001 C CNN
-	1    6500 4700
-	0    -1   -1   0
-$EndComp
 Wire Wire Line
 	6800 5200 6800 5600
-$Comp
-L 74xx:74LS161 U?
-U 1 1 5DB20441
-P 4200 4700
-F 0 "U?" V 4246 3856 50  0000 R CNN
-F 1 "74LS161" V 4155 3856 50  0000 R CNN
-F 2 "" H 4200 4700 50  0001 C CNN
-F 3 "http://www.ti.com/lit/gpn/sn74LS161" H 4200 4700 50  0001 C CNN
-	1    4200 4700
-	0    -1   -1   0
-$EndComp
 Connection ~ 4000 4200
 Wire Wire Line
@@
 Wire Wire Line
 	7750 2200 7750 5400
+$Comp
+L 74xx:74LS163 U?
+U 1 1 5E14CC07
+P 4200 4700
+AR Path="/5DCCFA8E/5E14CC07" Ref="U?"  Part="1"
+AR Path="/5D9B51E1/5E14CC07" Ref="U?"  Part="1"
+F 0 "U?" V 4246 3856 50  0000 R CNN
+F 1 "74LS163" V 4155 3856 50  0000 R CNN
+F 2 "" H 4200 4700 50  0001 C CNN
+F 3 "http://www.ti.com/lit/gpn/sn74LS163" H 4200 4700 50  0001 C CNN
+	1    4200 4700
+	0    -1   -1   0
+$EndComp
+$Comp
+L 74xx:74LS163 U?
+U 1 1 5E14E3D1
+P 6500 4700
+AR Path="/5DCCFA8E/5E14E3D1" Ref="U?"  Part="1"
+AR Path="/5D9B51E1/5E14E3D1" Ref="U?"  Part="1"
+F 0 "U?" V 6546 3856 50  0000 R CNN
+F 1 "74LS163" V 6455 3856 50  0000 R CNN
+F 2 "" H 6500 4700 50  0001 C CNN
+F 3 "http://www.ti.com/lit/gpn/sn74LS163" H 6500 4700 50  0001 C CNN
+	1    6500 4700
+	0    -1   -1   0
+$EndComp
 $EndSCHEMATC

Commit message: fixed labels
Parts:
- gave numbers to parts that had none: 7
Changed lines of the file:
@@
 $EndDescr
 $Comp
-L 74xx:74LS08 U?
+L 74xx:74LS08 U10
 U 1 1 5D9DAE24
 P 3800 2850
-F 0 "U?" V 3846 2670 50  0000 R CNN
+F 0 "U10" V 3846 2670 50  0000 R CNN
 F 1 "74LS08" V 3755 2670 50  0000 R CNN
 F 2 "" H 3800 2850 50  0001 C CNN
@@
 $EndComp
 $Comp
-L 74xx:74LS02 U?
+L 74xx:74LS02 U11
 U 1 1 5D9E5038
 P 3900 3450
-F 0 "U?" V 3946 3270 50  0000 R CNN
+F 0 "U11" V 3946 3270 50  0000 R CNN
 F 1 "74LS02" V 3855 3270 50  0000 R CNN
 F 2 "" H 3900 3450 50  0001 C CNN
@@
 	6200 3900 6200 4200
 $Comp
-L 74xx:74LS30 U?
+L 74xx:74LS30 U14
 U 1 1 5DA1D493
 P 5800 2500
-F 0 "U?" V 5846 2056 50  0000 R CNN
+F 0 "U14" V 5846 2056 50  0000 R CNN
 F 1 "74LS30" V 5755 2056 50  0000 R CNN
 F 2 "" H 5800 2500 50  0001 C CNN
@@
 $EndComp
 $Comp
-L 74xx:74LS04 U?
+L 74xx:74LS04 U1
 U 1 1 5DA24082
 P 4900 2800
-F 0 "U?" V 4946 2620 50  0000 R CNN
+F 0 "U1" V 4946 2620 50  0000 R CNN
 F 1 "74LS04" V 4855 2620 50  0000 R CNN
 F 2 "" H 4900 2800 50  0001 C CNN
@@
 $EndComp
 $Comp
-L 74xx:74LS04 U?
+L 74xx:74LS04 U1
 U 2 1 5DA25F00
 P 4900 3150
-F 0 "U?" V 4946 2970 50  0000 R CNN
+F 0 "U1" V 4946 2970 50  0000 R CNN
 F 1 "74LS04" V 4855 2970 50  0000 R CNN
 F 2 "" H 4900 3150 50  0001 C CNN
@@
 $EndComp
 $Comp
-L 74xx:74LS04 U?
+L 74xx:74LS04 U13
 U 3 1 5DA33E18
 P 4900 3500
-F 0 "U?" V 4946 3320 50  0000 R CNN
+F 0 "U13" V 4946 3320 50  0000 R CNN
 F 1 "74LS04" V 4855 3320 50  0000 R CNN
 F 2 "" H 4900 3500 50  0001 C CNN
@@
 $EndComp
 $Comp
-L 74xx:74LS04 U?
+L 74xx:74LS04 U1
 U 4 1 5DA35C5C
 P 4900 3900
-F 0 "U?" V 4946 3720 50  0000 R CNN
+F 0 "U1" V 4946 3720 50  0000 R CNN
 F 1 "74LS04" V 4855 3720 50  0000 R CNN
 F 2 "" H 4900 3900 50  0001 C CNN
@@
 Connection ~ 3800 4000
 $Comp
-L 74xx:74LS08 U?
+L 74xx:74LS08 U10
 U 2 1 5DB055E8
 P 6200 3450
-F 0 "U?" V 6246 3270 50  0000 R CNN
+F 0 "U10" V 6246 3270 50  0000 R CNN
 F 1 "74LS08" V 6155 3270 50  0000 R CNN
 F 2 "" H 6200 3450 50  0001 C CNN
@@
 P 4200 4700
 AR Path="/5DCCFA8E/5E14CC07" Ref="U?"  Part="1"
-AR Path="/5D9B51E1/5E14CC07" Ref="U?"  Part="1"
-F 0 "U?" V 4246 3856 50  0000 R CNN
+AR Path="/5D9B51E1/5E14CC07" Ref="U12"  Part="1"
+F 0 "U12" V 4246 3856 50  0000 R CNN
 F 1 "74LS163" V 4155 3856 50  0000 R CNN
 F 2 "" H 4200 4700 50  0001 C CNN
@@
 P 6500 4700
 AR Path="/5DCCFA8E/5E14E3D1" Ref="U?"  Part="1"
-AR Path="/5D9B51E1/5E14E3D1" Ref="U?"  Part="1"
-F 0 "U?" V 6546 3856 50  0000 R CNN
+AR Path="/5D9B51E1/5E14E3D1" Ref="U15"  Part="1"
+F 0 "U15" V 6546 3856 50  0000 R CNN
 F 1 "74LS163" V 6455 3856 50  0000 R CNN
 F 2 "" H 6500 4700 50  0001 C CNN

Commit message: finished hv sync
Parts:
- removed U1, U13: 74LS04, symbol 74xx:74LS04
- removed unit 2 of U10
- removed U11: 74LS02, symbol 74xx:74LS02
- removed U14: 74LS30, symbol 74xx:74LS30
- added unit 3 of U10
- added unit 4 of U10
- added U11, U3, U7: 74LS08, symbol 74xx:74LS08
- added U14: 74LS163, symbol 74xx:74LS163
- added U8: 74LS04, symbol 74xx:74LS04
- added U9: 74LS02, symbol 74xx:74LS02
- renumbered U15 to U13
Connections:
- net CP: no longer U13.2 (CP)
- net VCC: now also U12.10 (CET), U12.7 (CEP), U12.9 (~PE), U13.10 (CET), U13.7 (CEP), U13.9 (~PE), U14.10 (CET), U14.16 (VCC), U14.7 (CEP), U14.9 (~PE)
- net V_Blank: now also U7.13, U8.4
- net V_Sync: now also U7.11; no longer U10.3
- net at U10.1: now also U7.6; no longer U12.13 (Q1)
- net at U10.2: now also U10.8
- net at U12.12 (Q2): now also U7.2
- net at U12.11 (Q3): now also U11.12, U3.5
- net at U13.14 (Q0): now also U8.1
- net at U12.1 (~MR), U13.1 (~MR): now also U14.1 (~MR), U8.6
- net at U12.14 (Q0): now also U7.1
- net at U13.12 (Q2): now also U7.5
- net at U13.11 (Q3): now also U10.9
- net at U12.15 (TC): now also U13.2 (CP)
- net at U13.13 (Q1): now also U7.4
- net at U13.15 (TC): now also U14.2 (CP)
- net GND renamed Earth
- net Earth: now also U14.8 (GND)
- new net: U9.1, U9.5
- new net: U7.8, U9.2
- new net: U7.12, U9.3, U9.4
- new net: U10.11, U9.6
- new net: U8.3, U9.10
- new net: U10.3, U9.8
- new net: U11.13, U14.13 (Q1), U9.9
- new net: U10.10, U14.14 (Q0)
- new net: U10.12, U7.10, U8.2
- new net: U10.13, U3.6
- new net: U7.3, U7.9
- new net: U12.13 (Q1), U3.4
- new net: U11.11, U8.5
- no-connect marks 0 -> 15
Other:
- moved on the sheet: U12, U13
