File: breadboard-computer-video/breadboard-computer-video.sch (KiCad schematic (older format))
At the start: 19 parts, among them Q1 Q_NPN_BCE, Q2 Q_NPN_BCE, U4 74LS08, U5 74LS163, U6 74LS14, U7 28C256, U8 74LS02, Y1 12MHz

Commit message: finished hv sync
Parts:
- Y1: value 12MHz -> 6MHz
- gave numbers to parts that had none: 3
- renumbered U6 to U1, U8 to U2, U4 to U3, U7 to U6
Changed lines of the file:
@@
 $EndComp
 $Comp
-L 74xx:74LS02 U8
+L 74xx:74LS02 U2
 U 1 1 5D974F6E
 P 7300 2850
-F 0 "U8" H 7300 3175 50  0000 C CNN
+F 0 "U2" H 7300 3175 50  0000 C CNN
 F 1 "74LS02" H 7300 3084 50  0000 C CNN
 F 2 "" H 7300 2850 50  0001 C CNN
@@
 P 3600 2700
 F 0 "Y1" H 3600 2968 50  0000 C CNN
-F 1 "12MHz" H 3600 2877 50  0000 C CNN
+F 1 "6MHz" H 3600 2877 50  0000 C CNN
 F 2 "" H 3600 2700 50  0001 C CNN
 F 3 "https://www.mouser.com/datasheet/2/741/LFXTAL036736Bulk-998720.pdf" H 3600 2700 50  0001 C CNN
@@
 	4200 5200 3400 5200
 $Comp
-L 74xx:74LS08 U4
+L 74xx:74LS08 U3
 U 1 1 5DBCD2DA
 P 3300 6900
-F 0 "U4" V 3254 7088 50  0000 L CNN
+F 0 "U3" V 3254 7088 50  0000 L CNN
 F 1 "74LS08" V 3345 7088 50  0000 L CNN
 F 2 "" H 3300 6900 50  0001 C CNN
@@
 $EndSheet
 $Comp
-L Memory_EEPROM:28C256 U7
+L Memory_EEPROM:28C256 U6
 U 1 1 5E1F0F95
 P 4600 6100
-F 0 "U7" H 4600 7381 50  0000 C CNN
+F 0 "U6" H 4600 7381 50  0000 C CNN
 F 1 "28C256" H 4600 7290 50  0000 C CNN
 F 2 "" H 4600 6100 50  0001 C CNN
@@
 $EndComp
 $Comp
-L 74xx:74LS08 U4
+L 74xx:74LS08 U3
 U 3 1 5E99B421
 P 6700 3600
-F 0 "U4" H 6700 3925 50  0000 C CNN
+F 0 "U3" H 6700 3925 50  0000 C CNN
 F 1 "74LS08" H 6700 3834 50  0000 C CNN
 F 2 "" H 6700 3600 50  0001 C CNN
@@
 	6550 900  800  900
 $Comp
-L 74xx:74LS02 U8
+L 74xx:74LS02 U2
 U 2 1 5E9FFB0B
 P 6200 3050
-F 0 "U8" V 6154 3238 50  0000 L CNN
+F 0 "U2" V 6154 3238 50  0000 L CNN
 F 1 "74LS02" V 6245 3238 50  0000 L CNN
 F 2 "" H 6200 3050 50  0001 C CNN
@@
 $EndComp
 $Comp
-L 74xx:74LS14 U6
+L 74xx:74LS14 U1
 U 1 1 5EA1FAA0
 P 3600 1600
-F 0 "U6" H 3600 1917 50  0000 C CNN
+F 0 "U1" H 3600 1917 50  0000 C CNN
 F 1 "74LS14" H 3600 1826 50  0000 C CNN
 F 2 "" H 3600 1600 50  0001 C CNN
@@
 $EndComp
 $Comp
-L 74xx:74LS14 U6
+L 74xx:74LS14 U1
 U 2 1 5EA2147E
 P 4400 1600
-F 0 "U6" H 4400 1917 50  0000 C CNN
+F 0 "U1" H 4400 1917 50  0000 C CNN
 F 1 "74LS14" H 4400 1826 50  0000 C CNN
 F 2 "" H 4400 1600 50  0001 C CNN
@@
 $EndComp
 $Comp
-L 74xx:74LS02 U?
+L 74xx:74LS02 U2
 U 3 1 5DC8E486
 P 1950 6750
-F 0 "U?" V 1996 6570 50  0000 R CNN
+F 0 "U2" V 1996 6570 50  0000 R CNN
 F 1 "74LS02" V 1905 6570 50  0000 R CNN
 F 2 "" H 1950 6750 50  0001 C CNN
@@
 NoConn ~ 2950 5700
 $Comp
-L 74xx:74LS08 U?
+L 74xx:74LS08 U3
 U 4 1 5DCE6604
 P 3200 6300
-F 0 "U?" V 3154 6488 50  0000 L CNN
+F 0 "U3" V 3154 6488 50  0000 L CNN
 F 1 "74LS08" V 3245 6488 50  0000 L CNN
 F 2 "" H 3200 6300 50  0001 C CNN
@@
 	5000 5900 5750 5900
 $Comp
-L 74xx:74LS165 U?
+L 74xx:74LS165 U4
 U 1 1 5DD7AB27
 P 6250 4400
-F 0 "U?" V 6296 3356 50  0000 R CNN
+F 0 "U4" V 6296 3356 50  0000 R CNN
 F 1 "74LS165" V 6205 3356 50  0000 R CNN
 F 2 "" H 6250 4400 50  0001 C CNN
