File: video/VRAM.sch (KiCad schematic (older format))
At the start: 12 parts, among them U15 74LS08, U36 74LS04, U37 74LS08, U38 74LS273, U39 74LS245, U40 74LS04, U41 74LS243, U42 74LS243, U43 74LS245, U44 74LS245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

Commit message: Resize and plot video
Connections:
- net VCC is gone; now on net Earth: U38.10 (GND), U39.10 (GND), U41.13 (OEb), U41.7 (GND), U42.13 (OEb), U42.7 (GND), U43.10 (GND), U44.10 (GND), U45.10 (GND), U46.16 (GND), U46.22 (~CS1), U46.24 (~OE)
Other:
- moved on the sheet: U15B, U36B, U37A, U38, U39, U40A, U41, U42, U43, U44, U45, U46
