File: main/ALU-Add.sch (KiCad schematic (older format))
At the start: 6 parts, among them U37 74LS245, U38 74LS86, U39 74LS283, U40 74LS86, U41 74LS283, U42 74LS86

Commit message: Replot main with symbols
Parts:
- renumbered U37 to U36, U38 to U37, U39 to U38, U40 to U39, U41 to U40, U42 to U41
Changed lines of the file:
@@
 Sheet 10 26
 Title "ALU Adder/Subtractor"
-Date "2019-11-13"
+Date "2019-11-17"
 Rev "v1.0"
 Comp "Christopher Milan"
@@
 AR Path="/5E5B2E62/5D96F636" Ref="U?"  Part="1"
 AR Path="/5E5B2E62/5E0141CE/5D96F636" Ref="U?"  Part="1"
-AR Path="/5E5B2E62/5E0141CE/5D94D587/5D96F636" Ref="U38"  Part="1"
-F 0 "U38" H 3200 4933 50  0000 C CNN
+AR Path="/5E5B2E62/5E0141CE/5D94D587/5D96F636" Ref="U37"  Part="1"
+F 0 "U37" H 3200 4933 50  0000 C CNN
 F 1 "74LS86" H 3200 5024 50  0000 C CNN
 F 2 "" H 3200 5250 50  0001 C CNN
@@
 AR Path="/5E5B2E62/5D96F66E" Ref="U?"  Part="1"
 AR Path="/5E5B2E62/5E0141CE/5D96F66E" Ref="U?"  Part="1"
-AR Path="/5E5B2E62/5E0141CE/5D94D587/5D96F66E" Ref="U38"  Part="3"
-F 0 "U38" H 4300 4933 50  0000 C CNN
+AR Path="/5E5B2E62/5E0141CE/5D94D587/5D96F66E" Ref="U37"  Part="3"
+F 0 "U37" H 4300 4933 50  0000 C CNN
 F 1 "74LS86" H 4300 5024 50  0000 C CNN
 F 2 "" H 4300 5250 50  0001 C CNN
@@
 AR Path="/5E5B2E62/5D96F674" Ref="U?"  Part="1"
 AR Path="/5E5B2E62/5E0141CE/5D96F674" Ref="U?"  Part="1"
-AR Path="/5E5B2E62/5E0141CE/5D94D587/5D96F674" Ref="U38"  Part="2"
-F 0 "U38" H 3750 4933 50  0000 C CNN
+AR Path="/5E5B2E62/5E0141CE/5D94D587/5D96F674" Ref="U37"  Part="2"
+F 0 "U37" H 3750 4933 50  0000 C CNN
 F 1 "74LS86" H 3750 5024 50  0000 C CNN
 F 2 "" H 3750 5250 50  0001 C CNN
@@
 AR Path="/5E5B2E62/5D96F67A" Ref="U?"  Part="1"
 AR Path="/5E5B2E62/5E0141CE/5D96F67A" Ref="U?"  Part="1"
-AR Path="/5E5B2E62/5E0141CE/5D94D587/5D96F67A" Ref="U40"  Part="1"
-F 0 "U40" H 5400 4933 50  0000 C CNN
+AR Path="/5E5B2E62/5E0141CE/5D94D587/5D96F67A" Ref="U39"  Part="1"
+F 0 "U39" H 5400 4933 50  0000 C CNN
 F 1 "74LS86" H 5400 5024 50  0000 C CNN
 F 2 "" H 5400 5250 50  0001 C CNN
@@
 AR Path="/5E5B2E62/5D96F680" Ref="U?"  Part="1"
 AR Path="/5E5B2E62/5E0141CE/5D96F680" Ref="U?"  Part="1"
-AR Path="/5E5B2E62/5E0141CE/5D94D587/5D96F680" Ref="U38"  Part="4"
-F 0 "U38" H 4850 4933 50  0000 C CNN
+AR Path="/5E5B2E62/5E0141CE/5D94D587/5D96F680" Ref="U37"  Part="4"
+F 0 "U37" H 4850 4933 50  0000 C CNN
 F 1 "74LS86" H 4850 5024 50  0000 C CNN
 F 2 "" H 4850 5250 50  0001 C CNN
@@
 AR Path="/5E5B2E62/5D96F68F" Ref="U?"  Part="1"
 AR Path="/5E5B2E62/5E0141CE/5D96F68F" Ref="U?"  Part="1"
-AR Path="/5E5B2E62/5E0141CE/5D94D587/5D96F68F" Ref="U40"  Part="3"
-F 0 "U40" H 6500 4933 50  0000 C CNN
+AR Path="/5E5B2E62/5E0141CE/5D94D587/5D96F68F" Ref="U39"  Part="3"
+F 0 "U39" H 6500 4933 50  0000 C CNN
 F 1 "74LS86" H 6500 5024 50  0000 C CNN
 F 2 "" H 6500 5250 50  0001 C CNN
@@
 AR Path="/5E5B2E62/5D96F695" Ref="U?"  Part="1"
 AR Path="/5E5B2E62/5E0141CE/5D96F695" Ref="U?"  Part="1"
-AR Path="/5E5B2E62/5E0141CE/5D94D587/5D96F695" Ref="U40"  Part="2"
-F 0 "U40" H 5950 4933 50  0000 C CNN
+AR Path="/5E5B2E62/5E0141CE/5D94D587/5D96F695" Ref="U39"  Part="2"
+F 0 "U39" H 5950 4933 50  0000 C CNN
 F 1 "74LS86" H 5950 5024 50  0000 C CNN
 F 2 "" H 5950 5250 50  0001 C CNN
@@
 AR Path="/5E5B2E62/5D96F69B" Ref="U?"  Part="1"
 AR Path="/5E5B2E62/5E0141CE/5D96F69B" Ref="U?"  Part="1"
-AR Path="/5E5B2E62/5E0141CE/5D94D587/5D96F69B" Ref="U42"  Part="1"
-F 0 "U42" H 7600 4933 50  0000 C CNN
+AR Path="/5E5B2E62/5E0141CE/5D94D587/5D96F69B" Ref="U41"  Part="1"
+F 0 "U41" H 7600 4933 50  0000 C CNN
 F 1 "74LS86" H 7600 5024 50  0000 C CNN
 F 2 "" H 7600 5250 50  0001 C CNN
@@
 AR Path="/5E5B2E62/5D96F6A1" Ref="U?"  Part="1"
 AR Path="/5E5B2E62/5E0141CE/5D96F6A1" Ref="U?"  Part="1"
-AR Path="/5E5B2E62/5E0141CE/5D94D587/5D96F6A1" Ref="U40"  Part="4"
-F 0 "U40" H 7050 4933 50  0000 C CNN
+AR Path="/5E5B2E62/5E0141CE/5D94D587/5D96F6A1" Ref="U39"  Part="4"
+F 0 "U39" H 7050 4933 50  0000 C CNN
 F 1 "74LS86" H 7050 5024 50  0000 C CNN
 F 2 "" H 7050 5250 50  0001 C CNN
@@
 AR Path="/5E5B2E62/5D96F6BB" Ref="U?"  Part="1"
 AR Path="/5E5B2E62/5E0141CE/5D96F6BB" Ref="U?"  Part="1"
-AR Path="/5E5B2E62/5E0141CE/5D94D587/5D96F6BB" Ref="U39"  Part="1"
-F 0 "U39" H 4300 3019 50  0000 C CNN
+AR Path="/5E5B2E62/5E0141CE/5D94D587/5D96F6BB" Ref="U38"  Part="1"
+F 0 "U38" H 4300 3019 50  0000 C CNN
 F 1 "74LS283" H 4300 3110 50  0000 C CNN
 F 2 "" H 4300 4000 50  0001 C CNN
@@
 AR Path="/5E5B2E62/5D96F6C1" Ref="U?"  Part="1"
 AR Path="/5E5B2E62/5E0141CE/5D96F6C1" Ref="U?"  Part="1"
-AR Path="/5E5B2E62/5E0141CE/5D94D587/5D96F6C1" Ref="U41"  Part="1"
-F 0 "U41" H 6200 3019 50  0000 C CNN
+AR Path="/5E5B2E62/5E0141CE/5D94D587/5D96F6C1" Ref="U40"  Part="1"
+F 0 "U40" H 6200 3019 50  0000 C CNN
 F 1 "74LS283" H 6200 3110 50  0000 C CNN
 F 2 "" H 6200 4000 50  0001 C CNN
@@
 P 3150 2950
 AR Path="/5E5B2E62/5E1111DF" Ref="U?"  Part="1"
-AR Path="/5E5B2E62/5E0141CE/5D94D587/5E1111DF" Ref="U37"  Part="1"
-F 0 "U37" V 3196 2106 50  0000 R CNN
+AR Path="/5E5B2E62/5E0141CE/5D94D587/5E1111DF" Ref="U36"  Part="1"
+F 0 "U36" V 3196 2106 50  0000 R CNN
 F 1 "74LS245" V 3105 2106 50  0000 R CNN
 F 2 "" H 3150 2950 50  0001 C CNN
