File: main/ALU-L.sch (KiCad schematic (older format))
At the start: 14 parts, among them U22 74LS08, U23 74LS08, U24 74LS86, U25 74LS32, U26 74LS245, U27 74LS245, U28 74LS245, U29 74LS86, U30 74LS32, U32 74LS04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

Commit message: Replot main with symbols
Parts:
- gave numbers to parts that had none: 1
- renumbered U32 to U31, U33 to U32, U34 to U33, U36 to U35
Changed lines of the file:
@@
 Sheet 8 26
 Title "ALU Logic"
-Date "2019-11-13"
+Date "2019-11-17"
 Rev "v1.0"
 Comp "Christopher Milan"
@@
 $EndComp
 $Comp
-L 74xx:74LS245 U33
+L 74xx:74LS245 U32
 U 1 1 5EC634A5
 P 8050 3050
-F 0 "U33" H 8050 4031 50  0000 C CNN
+F 0 "U32" H 8050 4031 50  0000 C CNN
 F 1 "74LS245" H 8050 3940 50  0000 C CNN
 F 2 "" H 8050 3050 50  0001 C CNN
@@
 	7550 3700 10200 3700
 $Comp
-L 74xx:74LS245 U34
+L 74xx:74LS245 U33
 U 1 1 5F2CD1EA
 P 8050 4950
-F 0 "U34" H 8050 5931 50  0000 C CNN
+F 0 "U33" H 8050 5931 50  0000 C CNN
 F 1 "74LS245" H 8050 5840 50  0000 C CNN
 F 2 "" H 8050 4950 50  0001 C CNN
@@
 A_7
 $Comp
-L 74xx:74LS04 U32
+L 74xx:74LS04 U31
 U 1 1 5F4272AF
 P 7100 5700
-F 0 "U32" V 7146 5520 50  0000 R CNN
+F 0 "U31" V 7146 5520 50  0000 R CNN
 F 1 "74LS04" V 7055 5520 50  0000 R CNN
 F 2 "" H 7100 5700 50  0001 C CNN
@@
 $EndComp
 $Comp
-L 74xx:74LS04 U32
+L 74xx:74LS04 U31
 U 2 1 5F42D26C
 P 6750 5950
-F 0 "U32" V 6796 5770 50  0000 R CNN
+F 0 "U31" V 6796 5770 50  0000 R CNN
 F 1 "74LS04" V 6705 5770 50  0000 R CNN
 F 2 "" H 6750 5950 50  0001 C CNN
@@
 $EndComp
 $Comp
-L 74xx:74LS04 U32
+L 74xx:74LS04 U31
 U 3 1 5F455472
 P 7000 6550
-F 0 "U32" V 7046 6370 50  0000 R CNN
+F 0 "U31" V 7046 6370 50  0000 R CNN
 F 1 "74LS04" V 6955 6370 50  0000 R CNN
 F 2 "" H 7000 6550 50  0001 C CNN
@@
 $EndComp
 $Comp
-L 74xx:74LS04 U32
+L 74xx:74LS04 U31
 U 4 1 5F455478
 P 8200 6600
-F 0 "U32" V 8246 6420 50  0000 R CNN
+F 0 "U31" V 8246 6420 50  0000 R CNN
 F 1 "74LS04" V 8155 6420 50  0000 R CNN
 F 2 "" H 8200 6600 50  0001 C CNN
@@
 $EndComp
 $Comp
-L 74xx:74LS04 U32
+L 74xx:74LS04 U31
 U 5 1 5F46914B
 P 8450 6050
-F 0 "U32" V 8496 5870 50  0000 R CNN
+F 0 "U31" V 8496 5870 50  0000 R CNN
 F 1 "74LS04" V 8405 5870 50  0000 R CNN
 F 2 "" H 8450 6050 50  0001 C CNN
@@
 $EndComp
 $Comp
-L 74xx:74LS04 U32
+L 74xx:74LS04 U31
 U 6 1 5F469151
 P 9050 6150
-F 0 "U32" V 9096 5970 50  0000 R CNN
+F 0 "U31" V 9096 5970 50  0000 R CNN
 F 1 "74LS04" H 9005 5970 50  0000 R CNN
 F 2 "" H 9050 6150 50  0001 C CNN
@@
 $EndComp
 $Comp
-L 74xx:74LS04 U36
+L 74xx:74LS04 U35
 U 1 1 5F469157
 P 9600 6150
-F 0 "U36" V 9646 5970 50  0000 R CNN
+F 0 "U35" V 9646 5970 50  0000 R CNN
 F 1 "74LS04" H 9555 5970 50  0000 R CNN
 F 2 "" H 9600 6150 50  0001 C CNN
@@
 $EndComp
 $Comp
-L 74xx:74LS04 U36
+L 74xx:74LS04 U35
 U 2 1 5F46915D
 P 9250 5300
-F 0 "U36" V 9296 5120 50  0000 R CNN
+F 0 "U35" V 9296 5120 50  0000 R CNN
 F 1 "74LS04" V 9205 5120 50  0000 R CNN
 F 2 "" H 9250 5300 50  0001 C CNN
@@
 $EndComp
 $Comp
-L 74xx:74LS688 U?
+L 74xx:74LS688 U34
 U 1 1 5DAF0CC2
 P 8450 1950
-F 0 "U?" V 8404 706 50  0000 R CNN
+F 0 "U34" V 8404 706 50  0000 R CNN
 F 1 "74LS688" V 8495 706 50  0000 R CNN
 F 2 "" H 8450 1950 50  0001 C CNN
