File: main/Control-Logic.sch (KiCad schematic (older format))
At the start: 6 parts, among them U49 29F010-TSOP-SP, U50 74LS161, U51 29F010-TSOP-SP, U52 29F010-TSOP-SP, U53 29F010-TSOP-SP, U54 29F010-TSOP-SP

Commit message: Replot main with symbols
Parts:
- renumbered U49 to U48, U50 to U49, U51 to U50, U52 to U51, U53 to U52, U54 to U53
Changed lines of the file:
@@
 Sheet 12 26
 Title "Control Logic"
-Date "2019-11-13"
+Date "2019-11-17"
 Rev "v1.0"
 Comp "Christopher Milan"
@@
 DECSP
 $Comp
-L 74xx:74LS161 U50
+L 74xx:74LS161 U49
 U 1 1 5E8FB423
 P 2700 2000
-F 0 "U50" H 2700 2981 50  0000 C CNN
+F 0 "U49" H 2700 2981 50  0000 C CNN
 F 1 "74LS161" H 2700 2890 50  0000 C CNN
 F 2 "" H 2700 2000 50  0001 C CNN
@@
 	3200 1350 3200 1500
 $Comp
-L Memory_Flash:29F010-TSOP-SP U49
+L Memory_Flash:29F010-TSOP-SP U48
 U 1 1 5E904D82
 P 1800 4950
-F 0 "U49" H 1800 6331 50  0000 C CNN
+F 0 "U48" H 1800 6331 50  0000 C CNN
 F 1 "29F010-TSOP-SP" H 1800 6240 50  0000 C CNN
 F 2 "" H 1800 4950 50  0001 C CNN
@@
 	1700 5550 1700 6000
 $Comp
-L Memory_Flash:29F010-TSOP-SP U51
+L Memory_Flash:29F010-TSOP-SP U50
 U 1 1 5E93DAA5
 P 4500 4950
-F 0 "U51" H 4500 6331 50  0000 C CNN
+F 0 "U50" H 4500 6331 50  0000 C CNN
 F 1 "29F010-TSOP-SP" H 4500 6240 50  0000 C CNN
 F 2 "" H 4500 4950 50  0001 C CNN
@@
 	1000 4300 1000 4350
 $Comp
-L Memory_Flash:29F010-TSOP-SP U53
+L Memory_Flash:29F010-TSOP-SP U52
 U 1 1 5E9C71F9
 P 7200 4950
-F 0 "U53" H 7200 6331 50  0000 C CNN
+F 0 "U52" H 7200 6331 50  0000 C CNN
 F 1 "29F010-TSOP-SP" H 7200 6240 50  0000 C CNN
 F 2 "" H 7200 4950 50  0001 C CNN
@@
 	6450 1350 6450 900
 $Comp
-L Memory_Flash:29F010-TSOP-SP U52
+L Memory_Flash:29F010-TSOP-SP U51
 U 1 1 5EB0A972
 P 6550 1950
-F 0 "U52" H 6550 3331 50  0000 C CNN
+F 0 "U51" H 6550 3331 50  0000 C CNN
 F 1 "29F010-TSOP-SP" H 6550 3240 50  0000 C CNN
 F 2 "" H 6550 1950 50  0001 C CNN
@@
 	7350 2700 8000 2700
 $Comp
-L Memory_Flash:29F010-TSOP-SP U54
+L Memory_Flash:29F010-TSOP-SP U53
 U 1 1 5EC4C3F0
 P 9250 1950
-F 0 "U54" H 9250 3331 50  0000 C CNN
+F 0 "U53" H 9250 3331 50  0000 C CNN
 F 1 "29F010-TSOP-SP" H 9250 3240 50  0000 C CNN
 F 2 "" H 9250 1950 50  0001 C CNN
