File: main/F-Register.sch (KiCad schematic (older format))
At the start: 10 parts, among them U55 74LS245, U56 74LS173

Commit message: Replot main with symbols
Parts:
- renumbered U55 to U54, U56 to U55
Changed lines of the file:
@@
 Sheet 13 26
 Title "Flags Register"
-Date "2019-11-13"
+Date "2019-11-17"
 Rev "v1.0"
 Comp "Christopher Milan"
@@
 AR Path="/5D9E93FA/5DA6F82A" Ref="U?"  Part="1"
 AR Path="/5DA98D6D/5DA9AAB9/5DA6F82A" Ref="U?"  Part="1"
-AR Path="/5DA9DA3D/5DA6F82A" Ref="U56"  Part="1"
-F 0 "U56" V 7454 4494 50  0000 L CNN
+AR Path="/5DA9DA3D/5DA6F82A" Ref="U55"  Part="1"
+F 0 "U55" V 7454 4494 50  0000 L CNN
 F 1 "74LS173" V 7545 4494 50  0000 L CNN
 F 2 "" H 7500 3550 50  0001 C CNN
@@
 AR Path="/5D9E93FA/5DA6F7FD" Ref="U?"  Part="1"
 AR Path="/5DA98D6D/5DA9AAB9/5DA6F7FD" Ref="U?"  Part="1"
-AR Path="/5DA9DA3D/5DA6F7FD" Ref="U55"  Part="1"
-F 0 "U55" V 2946 2706 50  0000 R CNN
+AR Path="/5DA9DA3D/5DA6F7FD" Ref="U54"  Part="1"
+F 0 "U54" V 2946 2706 50  0000 R CNN
 F 1 "74LS245" V 2855 2706 50  0000 R CNN
 F 2 "" H 2900 3550 50  0001 C CNN
